File: Absolute_Encoder_Breakout/absolute_encoder_breakout/absolute_encoder_breakout.kicad_sch (KiCad schematic)
At the start: 1 part

Commit message: Main Board Schematic
Parts:
- added Conn1: Molex_SL_03, symbol MRDT_Connectors:Molex_SL_03
Connections:
- net 5V: no longer names the net of U1.1 (VDD5V)
- net 5V: now also Conn1.3
- net GND: no longer names the net of U1.4 (GND)
- net GND: now also Conn1.1
- net PWM: no longer names the net of U1.3 (OUT)
- net PWM: now also Conn1.2
Changed lines of the file:
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@@
 	(wire
 		(pts
-			(xy 107.95 78.74) (xy 128.27 78.74)
+			(xy 107.95 88.9) (xy 107.95 86.36)
 		)
 		(stroke
@@
 	(wire
 		(pts
-			(xy 107.95 93.98) (xy 128.27 93.98)
+			(xy 107.95 78.74) (xy 107.95 83.82)
 		)
 		(stroke
@@
 	(wire
 		(pts
-			(xy 107.95 88.9) (xy 128.27 88.9)
+			(xy 91.44 93.98) (xy 91.44 88.9)
 		)
 		(stroke
@@
 		)
 	)
-	(global_label "PWM"
-		(shape input)
-		(at 107.95 88.9 180)
+	(wire
+		(pts
+			(xy 128.27 93.98) (xy 91.44 93.98)
+		)
+		(stroke
+			(width 0)
+			(type default)
+		)
+	)
+	(wire
+		(pts
+			(xy 107.95 86.36) (xy 91.44 86.36)
+		)
+		(stroke
+			(width 0)
+			(type default)
+		)
+	)
+	(wire
+		(pts
+			(xy 107.95 83.82) (xy 91.44 83.82)
+		)
+		(stroke
+			(width 0)
+			(type default)
+		)
+	)
+	(wire
+		(pts
+			(xy 128.27 78.74) (xy 107.95 78.74)
+		)
+		(stroke
+			(width 0)
+			(type default)
+		)
+	)
+	(wire
+		(pts
+			(xy 128.27 88.9) (xy 107.95 88.9)
+		)
+		(stroke
+			(width 0)
+			(type default)
+		)
+	)
+	(symbol
+		(lib_id "MRDT_Connectors:Molex_SL_03")
+		(at 86.36 82.55 180)
+		(unit 1)
+		(exclude_from_sim no)
+		(in_bom yes)
+		(on_board yes)
+		(dnp no)
 		(fields_autoplaced yes)
-		(effects
-			(font
-				(size 1.27 1.27)
+		(property "Reference" "Conn1"
+			(at 85.09 77.47 0)
+			(effects
+				(font
+					(size 1.524 1.524)
+				)
 			)
-			(justify right)
 		)
-		(property "Intersheetrefs" "${INTERSHEET_REFS}"
-			(at 100.792 88.9 0)
+		(property "Value" "Molex_SL_03"
+			(at 85.09 80.01 0)
+			(effects
+				(font
+					(size 1.524 1.524)
+				)
+			)
+		)
+		(property "Footprint" ""
+			(at 86.36 82.55 0)
+			(effects
+				(font
+					(size 1.524 1.524)
+				)
+				(hide yes)
+			)
+		)
+		(property "Datasheet" ""
+			(at 86.36 82.55 0)
+			(effects
+				(font
+					(size 1.524 1.524)
+				)
+				(hide yes)
+			)
+		)
+		(property "Description" ""
+			(at 86.36 82.55 0)
 			(effects
 				(font
 					(size 1.27 1.27)
 				)
-				(justify right)
 				(hide yes)
 			)
 		)
-	)
-	(global_label "GND"
-		(shape input)
-		(at 107.95 93.98 180)
-		(fields_autoplaced yes)
-		(effects
-			(font
-				(size 1.27 1.27)
-			)
-			(justify right)
+		(pin "2"
 		)
-		(property "Intersheetrefs" "${INTERSHEET_REFS}"
-			(at 101.0943 93.98 0)
-			(effects
-				(font
-					(size 1.27 1.27)
+		(pin "3"
+		)
+		(pin "1"
+		)
+		(instances
+			(project ""
+				(path "/ebb075bd-427b-4233-b984-4ab8b040b824"
+					(reference "Conn1")
+					(unit 1)
 				)
-				(justify right)
-				(hide yes)
 			)
 		)
-	)
-	(global_label "5V"
-		(shape input)
-		(at 107.95 78.74 180)
-		(fields_autoplaced yes)
-		(effects
-			(font
-				(size 1.27 1.27)
-			)
-			(justify right)
-		)
-		(property "Intersheetrefs" "${INTERSHEET_REFS}"
-			(at 102.6667 78.74 0)
-			(effects
-				(font
-					(size 1.27 1.27)
-				)
-				(justify right)
-				(hide yes)
-			)
-		)
