File: Main_Board/Main_Board.kicad_sch (KiCad schematic)
At the start: 5 parts, among them U1 Teensy4.1_DEV-16771

Commit message: Schematic Finished
Connections:
- net PWM AE1 renamed AE1
- net PWM AE2 renamed AE2
- net PWM AE3 renamed AE3
- net PWM QE1-1 renamed QE1-1
- net PWM QE1-2 renamed QE1-2
- no-connect marks 0 -> 51
Changed lines of the file:
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@@
 	(generator_version "9.0")
 	(paper "A4")
+	(no_connect
+		(at 157.48 54.61)
+	)
+	(no_connect
+		(at 198.12 80.01)
+	)
+	(no_connect
+		(at 157.48 87.63)
+	)
+	(no_connect
+		(at 157.48 97.79)
+	)
+	(no_connect
+		(at 198.12 100.33)
+	)
+	(no_connect
+		(at 157.48 128.27)
+	)
+	(no_connect
+		(at 198.12 102.87)
+	)
+	(no_connect
+		(at 157.48 64.77)
+	)
+	(no_connect
+		(at 157.48 80.01)
+	)
+	(no_connect
+		(at 198.12 138.43)
+	)
+	(no_connect
+		(at 198.12 92.71)
+	)
+	(no_connect
+		(at 157.48 123.19)
+	)
+	(no_connect
+		(at 198.12 62.23)
+	)
+	(no_connect
+		(at 157.48 92.71)
+	)
+	(no_connect
+		(at 198.12 44.45)
+	)
+	(no_connect
+		(at 157.48 90.17)
+	)
+	(no_connect
+		(at 198.12 115.57)
+	)
+	(no_connect
+		(at 198.12 118.11)
+	)
+	(no_connect
+		(at 198.12 120.65)
+	)
+	(no_connect
+		(at 157.48 77.47)
+	)
+	(no_connect
+		(at 157.48 100.33)
+	)
+	(no_connect
+		(at 198.12 64.77)
+	)
+	(no_connect
+		(at 198.12 95.25)
+	)
+	(no_connect
+		(at 157.48 105.41)
+	)
+	(no_connect
+		(at 157.48 72.39)
+	)
+	(no_connect
+		(at 198.12 49.53)
+	)
+	(no_connect
+		(at 157.48 62.23)
+	)
+	(no_connect
+		(at 198.12 59.69)
+	)
+	(no_connect
+		(at 157.48 57.15)
+	)
+	(no_connect
+		(at 157.48 74.93)
+	)
+	(no_connect
+		(at 198.12 123.19)
+	)
+	(no_connect
+		(at 157.48 69.85)
+	)
+	(no_connect
+		(at 157.48 125.73)
+	)
+	(no_connect
+		(at 198.12 72.39)
+	)
+	(no_connect
+		(at 198.12 130.81)
+	)
+	(no_connect
+		(at 198.12 69.85)
+	)
+	(no_connect
+		(at 198.12 77.47)
+	)
+	(no_connect
+		(at 157.48 82.55)
+	)
+	(no_connect
+		(at 198.12 57.15)
+	)
+	(no_connect
+		(at 198.12 110.49)
+	)
+	(no_connect
+		(at 198.12 90.17)
+	)
+	(no_connect
+		(at 198.12 46.99)
+	)
+	(no_connect
+		(at 198.12 125.73)
+	)
+	(no_connect
+		(at 157.48 130.81)
+	)
+	(no_connect
+		(at 157.48 102.87)
+	)
+	(no_connect
+		(at 198.12 85.09)
+	)
+	(no_connect
+		(at 198.12 82.55)
+	)
+	(no_connect
+		(at 198.12 113.03)
+	)
+	(no_connect
+		(at 198.12 54.61)
+	)
+	(no_connect
+		(at 157.48 85.09)
+	)
+	(no_connect
+		(at 198.12 128.27)
+	)
 	(wire
 		(pts
@@
 	(wire
 		(pts
-			(xy 143.51 72.39) (xy 143.51 69.85)
+			(xy 143.51 73.66) (xy 143.51 69.85)
 		)
 		(stroke
@@
 	(wire
 		(pts
+			(xy 198.12 41.91) (xy 208.28 41.91)
+		)
+		(stroke
+			(width 0)
+			(type default)
+		)
+	)
+	(wire
+		(pts
 			(xy 139.7 69.85) (xy 139.7 72.39)
 		)
@@
 	(wire
 		(pts
+			(xy 208.28 41.91) (xy 208.28 34.29)
+		)
+		(stroke
+			(width 0)
+			(type default)
+		)
+	)
+	(wire
+		(pts
 			(xy 128.27 69.85) (xy 125.73 69.85)
 		)
@@
 	(wire
 		(pts
-			(xy 198.12 41.91) (xy 203.2 41.91)
-		)
-		(stroke
-			(width 0)
-			(type default)
-		)
-	)
-	(wire
-		(pts
 			(xy 143.51 69.85) (xy 139.7 69.85)
 		)
@@
 		)
 	)
-	(global_label "PWM AE2"
+	(global_label "AE2"
 		(shape input)
 		(at 148.59 113.03 180)
@@
 		)
 		(property "Intersheetrefs" "${INTERSHEET_REFS}"
-			(at 137.0173 113.03 0)
+			(at 142.1577 113.03 0)
 			(effects
 				(font
@@
 		)
 	)
-	(global_label "PWM QE1-2"
-		(shape input)
+	(global_label "QE1-2"
+		(shape output)
 		(at 95.25 66.04 90)
 		(fields_autoplaced yes)
@@
 		)
 		(property "Intersheetrefs" "${INTERSHEET_REFS}"
-			(at 95.25 51.4435 90)
+			(at 95.25 56.5839 90)
 			(effects
 				(font
@@
 		)
 	)
-	(global_label "PWM AE2"
-		(shape input)
+	(global_label "AE2"
+		(shape output)
 		(at 123.19 66.04 90)
 		(fields_autoplaced yes)
@@
 		)
 		(property "Intersheetrefs" "${INTERSHEET_REFS}"
-			(at 123.19 54.4673 90)
+			(at 123.19 59.6077 90)
 			(effects
 				(font
@@
 		)
 	)
-	(global_label "PWM QE1-1"
-		(shape input)
+	(global_label "QE1-1"
+		(shape output)
 		(at 92.71 66.04 90)
 		(fields_autoplaced yes)
@@
 		)
 		(property "Intersheetrefs" "${INTERSHEET_REFS}"
-			(at 92.71 51.4435 90)
+			(at 92.71 56.5839 90)
 			(effects
 				(font
@@
 		)
 	)
-	(global_label "PWM AE3"
-		(shape input)
+	(global_label "AE3"
+		(shape output)
 		(at 107.95 66.04 90)
 		(fields_autoplaced yes)
@@
 		)
 		(property "Intersheetrefs" "${INTERSHEET_REFS}"
-			(at 107.95 54.4673 90)
+			(at 107.95 59.6077 90)
 			(effects
 				(font
@@
 		)
 	)
-	(global_label "PWM QE1-2"
+	(global_label "QE1-2"
 		(shape input)
 		(at 148.59 120.65 180)
@@
 		)
 		(property "Intersheetrefs" "${INTERSHEET_REFS}"
-			(at 133.9935 120.65 0)
+			(at 139.1339 120.65 0)
 			(effects
 				(font
@@
 		)
 	)
-	(global_label "PWM AE1"
-		(shape input)
+	(global_label "AE1"
+		(shape output)
 		(at 137.16 66.04 90)
 		(fields_autoplaced yes)
@@
 		)
 		(property "Intersheetrefs" "${INTERSHEET_REFS}"
-			(at 137.16 54.4673 90)
+			(at 137.16 59.6077 90)
 			(effects
 				(font
@@
 		)
 	)
-	(global_label "PWM AE1"
+	(global_label "AE1"
 		(shape input)
 		(at 148.59 110.49 180)
@@
 		)
 		(property "Intersheetrefs" "${INTERSHEET_REFS}"
-			(at 137.0173 110.49 0)
+			(at 142.1577 110.49 0)
 			(effects
 				(font
@@
 		)
 	)
-	(global_label "PWM AE3"
+	(global_label "AE3"
 		(shape input)
 		(at 148.59 115.57 180)
@@
 		)
 		(property "Intersheetrefs" "${INTERSHEET_REFS}"
-			(at 137.0173 115.57 0)
+			(at 142.1577 115.57 0)
 			(effects
 				(font
@@
 		)
 	)
-	(global_label "PWM QE1-1"
+	(global_label "QE1-1"
 		(shape input)
 		(at 148.59 118.11 180)
@@
 		)
 		(property "Intersheetrefs" "${INTERSHEET_REFS}"
-			(at 133.9935 118.11 0)
+			(at 139.1339 118.11 0)
 			(effects
 				(font
@@
 	(symbol
 		(lib_id "power:GND")
-		(at 143.51 72.39 0)
+		(at 143.51 73.66 0)
 		(unit 1)
 		(exclude_from_sim no)
@@
 		(fields_autoplaced yes)
 		(property "Reference" "#PWR06"
+			(at 143.51 80.01 0)
+			(effects
+				(font
+					(size 1.27 1.27)
+				)
+				(hide yes)
+			)
+		)
+		(property "Value" "GND"
 			(at 143.51 78.74 0)
 			(effects
@@
 					(size 1.27 1.27)
 				)
-				(hide yes)
-			)
-		)
-		(property "Value" "GND"
-			(at 143.51 77.47 0)
-			(effects
-				(font
-					(size 1.27 1.27)
-				)
 			)
 		)
 		(property "Footprint" ""
-			(at 143.51 72.39 0)
+			(at 143.51 73.66 0)
 			(effects
 				(font
@@
 		)
 		(property "Datasheet" ""
-			(at 143.51 72.39 0)
+			(at 143.51 73.66 0)
 			(effects
 				(font
@@
 		)
 		(property "Description" "Power symbol creates a global label with name \"GND\" , ground"
-			(at 143.51 72.39 0)
+			(at 143.51 73.66 0)
 			(effects
 				(font
@@
 	(symbol
 		(lib_id "power:+5V")
-		(at 203.2 41.91 0)
+		(at 208.28 34.29 0)
 		(unit 1)
 		(exclude_from_sim no)
@@
 		(fields_autoplaced yes)
 		(property "Reference" "#PWR05"
-			(at 203.2 45.72 0)
+			(at 208.28 38.1 0)
 			(effects
 				(font
@@
 		)
 		(property "Value" "+5V"
-			(at 203.2 36.83 0)
+			(at 208.28 29.21 0)
 			(effects
 				(font
@@
 		)
 		(property "Footprint" ""
-			(at 203.2 41.91 0)
+			(at 208.28 34.29 0)
 			(effects
 				(font
@@
 		)
 		(property "Datasheet" ""
-			(at 203.2 41.91 0)
+			(at 208.28 34.29 0)
 			(effects
 				(font
@@
 		)
 		(property "Description" "Power symbol creates a global label with name \"+5V\""
-			(at 203.2 41.91 0)
-			(effects
-				(font
+			(at 208.28 34.29 0)
+			(effects
+				(font
