File: encoder_breakout/absolute_encoder_breakout/absolute_encoder_breakout.kicad_sch (KiCad schematic)
At the start: 4 parts

Commit message: Final Encoder Breakout
Parts:
- removed Conn1: Molex_SL_03, Connector_JST:JST_PH_B3B-PH-K_1x03_P2.00mm_Vertical, symbol MRDT_Connectors:Molex_SL_03
- added J1: Conn_01x03_Pin, Connector_JST:JST_PH_S3B-PH-K_1x03_P2.00mm_Horizontal, symbol Connector:Conn_01x03_Pin
- C1: footprint (none) -> Capacitor_SMD:C_0603_1608Metric_Pad1.08x0.95mm_HandSolder
Connections:
- net GND: now also J1.3 (Pin_3)
- net at C1.1, R1.1, U1.1 (VDD5V)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: now also J1.1 (Pin_1)
- net at U1.3 (OUT): now also J1.2 (Pin_2)
Changed lines of the file:
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@@
 			)
 		)
-		(property "Footprint" ""
+		(property "Footprint" "Capacitor_SMD:C_0603_1608Metric_Pad1.08x0.95mm_HandSolder"
 			(at 115.2652 92.71 0)
 			(effects
@@
 	)
 	(symbol
-		(lib_id "MRDT_Connectors:Molex_SL_03")
-		(at 100.33 82.55 180)
+		(lib_id "Connector:Conn_01x03_Pin")
+		(at 100.33 86.36 0)
 		(unit 1)
 		(exclude_from_sim no)
@@
 		(dnp no)
 		(fields_autoplaced yes)
-		(property "Reference" "Conn1"
-			(at 99.06 77.47 0)
+		(property "Reference" "J1"
+			(at 100.965 78.74 0)
 			(effects
 				(font
-					(size 1.524 1.524)
+					(size 1.27 1.27)
 				)
 			)
 		)
-		(property "Value" "Molex_SL_03"
-			(at 99.06 80.01 0)
+		(property "Value" "Conn_01x03_Pin"
+			(at 100.965 81.28 0)
 			(effects
 				(font
-					(size 1.524 1.524)
+					(size 1.27 1.27)
 				)
 			)
 		)
-		(property "Footprint" "Connector_JST:JST_PH_B3B-PH-K_1x03_P2.00mm_Vertical"
-			(at 100.33 82.55 0)
-			(effects
-				(font
-					(size 1.524 1.524)
-				)
-				(hide yes)
-			)
-		)
-		(property "Datasheet" ""
-			(at 100.33 82.55 0)
-			(effects
-				(font
-					(size 1.524 1.524)
-				)
-				(hide yes)
-			)
-		)
-		(property "Description" ""
-			(at 100.33 82.55 0)
+		(property "Footprint" "Connector_JST:JST_PH_S3B-PH-K_1x03_P2.00mm_Horizontal"
+			(at 100.33 86.36 0)
 			(effects
 				(font
@@
 			)
 		)
-		(pin "2"
+		(property "Datasheet" "~"
+			(at 100.33 86.36 0)
+			(effects
+				(font
+					(size 1.27 1.27)
+				)
+				(hide yes)
+			)
+		)
+		(property "Description" "Generic connector, single row, 01x03, script generated"
+			(at 100.33 86.36 0)
+			(effects
+				(font
+					(size 1.27 1.27)
+				)
+				(hide yes)
+			)
 		)
 		(pin "3"
@@
 		(pin "1"
 		)
+		(pin "2"
+		)
 		(instances
 			(project ""
 				(path "/ebb075bd-427b-4233-b984-4ab8b040b824"
-					(reference "Conn1")
+					(reference "J1")
 					(unit 1)
 				)
