File: board/Main_Board.kicad_pcb (KiCad board)
At the start: 2 copper layers, 61.5 x 34.8 mm, 24 parts, among them J2 J2 Encoder, J3 J3 Encoder, J4 J4 Encoder, J5 Pitch Encoder, J6 FWD Conn_01x02_Pin, J6 RVS Conn_01x02_Pin, U1 Teensy4.1_DEV-16771

Commit message: Add plated mounting holes
Parts:
- removed sign: LOGO, LOGO
- H1: renamed from H2; footprint MRDT_Drill_Holes:4_40_Hole -> MRDT_Drill_Holes:4_40_Hole_Pad_Via
- H2, H3: footprint MRDT_Drill_Holes:4_40_Hole -> MRDT_Drill_Holes:4_40_Hole_Pad_Via
- H4: renamed from H3; footprint MRDT_Drill_Holes:4_40_Hole -> MRDT_Drill_Holes:4_40_Hole_Pad_Via
- J1: renamed from G FWD
- J7: renamed from G RVS
- J8: renamed from J6 FWD
- J9: renamed from J6 RVS
- SW1: renamed from ON     OFF
- moved C1 8.48 mm to (122.7, 79.5), turned to 0 degrees
- renumbered X to J6
Connections:
- SW1 pad : GND -> (no net)
Routing:
- net +3V3: track 93.3 -> 83.7 mm

Commit message: Final design files as ordered
Parts:
- moved C1 0.51 mm to (122.7, 80.0)
- moved D1 0.38 mm to (136.7, 70.0)
- moved D3 0.38 mm to (139.2, 70.0)
Routing:
- net +3V3: track 83.7 -> 84.2 mm
- net GND: vias 30 -> 31
Changed lines of the file:
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@@
 			(outputformat 1)
 			(mirror no)
-			(drillshape 1)
+			(drillshape 0)
 			(scaleselection 1)
-			(outputdirectory "")
+			(outputdirectory "MiniArm_Gerbs/")
 		)
 	)
@@
 	(footprint "LED_SMD:LED_0603_1608Metric_Pad1.05x0.95mm_HandSolder"
 		(layer "F.Cu")
-		(at 139.192 69.596 -90)
+		(at 139.192 69.977 -90)
 		(descr "LED SMD 0603 (1608 Metric), square (rectangular) end terminal, IPC-7351 nominal, (Body size source: http://www.tortai-tech.com/upload/download/2011102023233369053.pdf), generated with kicad-footprint-generator")
 		(tags "LED handsolder")
@@
 	(footprint "LED_SMD:LED_0603_1608Metric_Pad1.05x0.95mm_HandSolder"
 		(layer "F.Cu")
-		(at 136.652 69.596 -90)
+		(at 136.652 69.977 -90)
 		(descr "LED SMD 0603 (1608 Metric), square (rectangular) end terminal, IPC-7351 nominal, (Body size source: http://www.tortai-tech.com/upload/download/2011102023233369053.pdf), generated with kicad-footprint-generator")
 		(tags "LED handsolder")
@@
 	(footprint "Capacitor_SMD:C_0603_1608Metric_Pad1.08x0.95mm_HandSolder"
 		(layer "F.Cu")
-		(at 122.7328 79.502)
+		(at 122.7328 80.01)
 		(descr "Capacitor SMD 0603 (1608 Metric), square (rectangular) end terminal, IPC-7351 nominal with elongated pad for handsoldering. (Body size source: IPC-SM-782 page 76, https://www.pcb-3d.com/wordpress/wp-content/uploads/ipc-sm-782a_amendment_1_and_2.pdf), generated with kicad-footprint-generator")
 		(tags "capacitor handsolder")
@@
 	)
 	(via
+		(at 124.714 80.01)
+		(size 0.6)
+		(drill 0.3)
+		(layers "F.Cu" "B.Cu")
+		(free yes)
+		(net 1)
+	)
+	(via
 		(at 154.686 71.12)
 		(size 0.6)
@@
 	)
 	(segment
-		(start 121.8703 79.502)
-		(end 121.8703 77.5197)
-		(width 0.2)
+		(start 152.4 96.774)
+		(end 152.908 96.774)
+		(width 0.254)
 		(layer "F.Cu")
 		(net 2)
@@
 	)
 	(segment
-		(start 153.226 97.6)
-		(end 152.4 96.774)
-		(width 0.254)
-		(layer "F.Cu")
-		(net 2)
-	)
-	(segment
 		(start 127.286 70.072)
 		(end 127.286 73.5245)
@@
 	)
 	(segment
-		(start 121.8703 77.5197)
-		(end 121.92 77.47)
-		(width 0.2)
-		(layer "F.Cu")
-		(net 2)
-	)
-	(segment
 		(start 146.812 96.774)
 		(end 145.034 96.774)
@@
 	(segment
 		(start 152.4 92.71)
-		(end 152.4 96.774)
+		(end 152.4 96.266)
 		(width 0.254)
 		(layer "F.Cu")
@@
 	)
 	(segment
+		(start 152.4 96.266)
+		(end 152.908 96.774)
+		(width 0.254)
+		(layer "F.Cu")
+		(net 2)
+	)
+	(segment
+		(start 121.8703 77.5197)
+		(end 121.92 77.47)
+		(width 0.2)
+		(layer "F.Cu")
+		(net 2)
+	)
+	(segment
 		(start 125.762 97.758)
 		(end 125.762 99.018)
@@
 	)
 	(segment
+		(start 153.226 97.092)
+		(end 152.908 96.774)
+		(width 0.254)
+		(layer "F.Cu")
+		(net 2)
+	)
+	(segment
 		(start 137.668 96.774)
 		(end 126.746 96.774)
@@
 	)
 	(segment
-		(start 153.226 99.06)
-		(end 153.226 97.6)
-		(width 0.254)
+		(start 121.8703 80.01)
+		(end 121.8703 77.5197)
+		(width 0.2)
 		(layer "F.Cu")
 		(net 2)
@@
 	)
 	(segment
-		(start 152.4 96.774)
+		(start 153.226 99.06)
+		(end 153.226 97.092)
+		(width 0.254)
+		(layer "F.Cu")
+		(net 2)
+	)
+	(segment
+		(start 152.908 96.774)
 		(end 156.464 96.774)
 		(width 0.254)
@@
 	)
 	(segment
-		(start 136.652 70.471)
+		(start 136.652 70.852)
 		(end 136.652 72.4935)
 		(width 0.2)
@@
 	(segment
 		(start 139.192 72.4935)
-		(end 139.192 70.471)
+		(end 139.192 70.852)
 		(width 0.2)
 		(layer "F.Cu")
@@
 			)
 		)
+	)
+	(zone
+		(net 0)
+		(net_name "")
+		(layers "*.Mask")
+		(hatch edge 0.5)
+		(connect_pads
+			(clearance 0)
+		)
+		(min_thickness 0.25)
+		(filled_areas_thickness no)
+		(fill yes
+			(thermal_gap 0.5)
+			(thermal_bridge_width 0.5)
+		)
+		(polygon
+			(pts
+				(xy 172.778653 66.397355) (xy 173.155938 66.414798) (xy 173.272743 66.425622) (xy 173.64681 66.477802)
+				(xy 173.762119 66.499357) (xy 174.129775 66.585829) (xy 174.242603 66.617931) (xy 174.600712 66.737957)
+				(xy 174.710096 66.780332) (xy 175.055603 66.932888) (xy 175.160612 66.985177) (xy 175.490569 67.168962)
+				(xy 175.590305 67.230716) (xy 175.901897 67.444162) (xy 175.995506 67.514851) (xy 176.286075 67.756135)
+				(xy 176.372768 67.835166) (xy 176.639834 68.102232) (xy 176.718865 68.188925) (xy 176.960149 68.479494)
+				(xy 177.030838 68.573103) (xy 177.244284 68.884695) (xy 177.306038 68.984431) (xy 177.489823 69.314388)
+				(xy 177.542112 69.419397) (xy 177.694668 69.764904) (xy 177.737043 69.874288) (xy 177.857069 70.232397)
+				(xy 177.889171 70.345225) (xy 177.975643 70.712881) (xy 177.997198 70.82819) (xy 178.049378 71.202257)
+				(xy 178.060202 71.319062) (xy 178.077645 71.696347) (xy 178.079 71.755) (xy 178.079 98.425) (xy 178.077645 98.483653)
+				(xy 178.060202 98.860938) (xy 178.049378 98.977743) (xy 177.997198 99.35181) (xy 177.975643 99.467119)
+				(xy 177.889171 99.834775) (xy 177.857069 99.947603) (xy 177.737043 100.305712) (xy 177.694668 100.415096)
+				(xy 177.542112 100.760603) (xy 177.489823 100.865612) (xy 177.306038 101.195569) (xy 177.244284 101.295305)
+				(xy 177.030838 101.606897) (xy 176.960149 101.700506) (xy 176.718865 101.991075) (xy 176.639834 102.077768)
+				(xy 176.372768 102.344834) (xy 176.286075 102.423865) (xy 175.995506 102.665149) (xy 175.901897 102.735838)
+				(xy 175.590305 102.949284) (xy 175.490569 103.011038) (xy 175.160612 103.194823) (xy 175.055603 103.247112)
+				(xy 174.710096 103.399668) (xy 174.600712 103.442043) (xy 174.242603 103.562069) (xy 174.129775 103.594171)
+				(xy 173.762119 103.680643) (xy 173.64681 103.702198) (xy 173.272743 103.754378) (xy 173.155938 103.765202)
+				(xy 172.778653 103.782645) (xy 172.72 103.784) (xy 119.38 103.784) (xy 119.321347 103.782645) (xy 118.944062 103.765202)
+				(xy 118.827257 103.754378) (xy 118.45319 103.702198) (xy 118.337881 103.680643) (xy 117.970225 103.594171)
+				(xy 117.857397 103.562069) (xy 117.499288 103.442043) (xy 117.389904 103.399668) (xy 117.044397 103.247112)
+				(xy 116.939388 103.194823) (xy 116.609431 103.011038) (xy 116.509695 102.949284) (xy 116.198103 102.735838)
+				(xy 116.104494 102.665149) (xy 115.813925 102.423865) (xy 115.727232 102.344834) (xy 115.460166 102.077768)
+				(xy 115.381135 101.991075) (xy 115.139851 101.700506) (xy 115.069162 101.606897) (xy 114.855716 101.295305)
+				(xy 114.793962 101.195569) (xy 114.610177 100.865612) (xy 114.557888 100.760603) (xy 114.405332 100.415096)
+				(xy 114.362957 100.305712) (xy 114.242931 99.947603) (xy 114.210829 99.834775) (xy 114.124357 99.467119)
+				(xy 114.102802 99.35181) (xy 114.050622 98.977743) (xy 114.039798 98.860938) (xy 114.022355 98.483653)
+				(xy 114.021 98.425) (xy 114.021 71.755) (xy 114.022355 71.696347) (xy 114.039798 71.319062) (xy 114.050622 71.202257)
+				(xy 114.102802 70.82819) (xy 114.124357 70.712881) (xy 114.210829 70.345225) (xy 114.242931 70.232397)
+				(xy 114.362957 69.874288) (xy 114.405332 69.764904) (xy 114.557888 69.419397) (xy 114.610177 69.314388)
+				(xy 114.793962 68.984431) (xy 114.855716 68.884695) (xy 115.069162 68.573103) (xy 115.139851 68.479494)
+				(xy 115.381135 68.188925) (xy 115.460166 68.102232) (xy 115.727232 67.835166) (xy 115.813925 67.756135)
+				(xy 116.104494 67.514851) (xy 116.198103 67.444162) (xy 116.509695 67.230716) (xy 116.609431 67.168962)
+				(xy 116.939388 66.985177) (xy 117.044397 66.932888) (xy 117.389904 66.780332) (xy 117.499288 66.737957)
+				(xy 117.857397 66.617931) (xy 117.970225 66.585829) (xy 118.337881 66.499357) (xy 118.45319 66.477802)
+				(xy 118.827257 66.425622) (xy 118.944062 66.414798) (xy 119.321347 66.397355) (xy 119.38 66.396)
+				(xy 172.72 66.396)
+			)
+		)
+		(polygon
+			(pts
+				(xy 141.097 68.986) (xy 140.335 67.564) (xy 123.698117 67.564) (xy 122.9614 68.9864) (xy 119.251981 68.986)
+				(xy 118.997036 69.009624) (xy 118.745357 69.05667) (xy 118.499101 69.126737) (xy 118.260342 69.219232)
+				(xy 118.031154 69.333354) (xy 117.813467 69.46814) (xy 117.609144 69.622438) (xy 117.41993 69.79493)
+				(xy 117.247438 69.984144) (xy 117.09314 70.188467) (xy 116.958354 70.406154) (xy 116.844232 70.635342)
+				(xy 116.751737 70.874101) (xy 116.68167 71.120357) (xy 116.634624 71.372036) (xy 116.611 71.62698)
+				(xy 116.611 75.692) (xy 115.316 76.454) (xy 115.316 93.98) (xy 116.586 94.996) (xy 116.611 98.553019)
+				(xy 116.634624 98.807963) (xy 116.68167 99.059642) (xy 116.751737 99.305898) (xy 116.844232 99.544657)
+				(xy 116.958354 99.773845) (xy 117.09314 99.991532) (xy 117.247438 100.195855) (xy 117.41993 100.385069)
+				(xy 117.609144 100.557561) (xy 117.813467 100.711859) (xy 118.031154 100.846645) (xy 118.260342 100.960767)
+				(xy 118.499101 101.053262) (xy 118.745357 101.123329) (xy 118.997036 101.170375) (xy 119.251981 101.194)
+				(xy 172.848019 101.194) (xy 173.102963 101.170375) (xy 173.354642 101.123329) (xy 173.600898 101.053262)
+				(xy 173.839657 100.960767) (xy 174.068845 100.846645) (xy 174.286532 100.711859) (xy 174.490855 100.557561)
+				(xy 174.680069 100.385069) (xy 174.852561 100.195855) (xy 175.006859 99.991532) (xy 175.141645 99.773845)
+				(xy 175.255767 99.544657) (xy 175.348262 99.305898) (xy 175.418329 99.059642) (xy 175.465375 98.807963)
+				(xy 175.489 98.553019) (xy 175.514 94.996) (xy 176.784 93.98) (xy 176.784 76.454) (xy 175.489 75.692)
+				(xy 175.489 71.62698) (xy 175.465375 71.372036) (xy 175.418329 71.120357) (xy 175.348262 70.874101)
+				(xy 175.255767 70.635342) (xy 175.141645 70.406154) (xy 175.006859 70.188467) (xy 174.852561 69.984144)
+				(xy 174.680069 69.79493) (xy 174.490855 69.622438) (xy 174.286532 69.46814) (xy 174.068845 69.333354)
+				(xy 173.839657 69.219232) (xy 173.600898 69.126737) (xy 173.354642 69.05667) (xy 173.102963 69.009624)
+				(xy 172.848019 68.986)
+			)
+		)
